File: pcb/PicoSax/Backup/260114 PicoSax/PicoSax.kicad_sch (KiCad schematic)
At the start: 75 parts, among them J3 Conn_01x02, SW8va1 Gateron_KS-33, SW8vb1 Gateron_KS-33, U1 Perfboard

Commit message: KS-33 Update
Routing still required.  If wanting to work on previous version, see Backup.
Parts:
- removed C4: 0.1uF, Capacitor_SMD:C_0805_2012Metric_Pad1.18x1.45mm_HandSolder, symbol PicoSax:C
- removed D2: 19-C47/RSGHBHC-5V01/2T, PicoSax:19-C47_RSGHBHC-5V01-2T, symbol PicoSax:19-C47_RSGHBHC-5V01_2T
- removed SW8va1, SW8vb1, SWA1, SWB1, SWBb1, SWC1, SWCtrl1, SWD1, SWDup1, SWE1, SWEb1, SWF1, SWG1, SWGs1, SWSpr1: Gateron_KS-33, PicoSax:KS-33, symbol PicoSax:Gateron_KS-33
- added SW8va1, SW8vb1, SWA1, SWB1, SWBb1, SWC1, SWCTRL1, SWD1, SWDup1, SWE1, SWEb1, SWF1, SWG1, SWGs1, SWSPR1: Omron_B3K_L13L, MyLibrary:Omron B3K L13L, symbol PicoSax:Omron_B3K_L13L
- renumbered C11 to C10, C12 to C11, C13 to C12, C14 to C13, C15 to C14, C16 to C15, C17 to C16, C18 to C17, C5 to C4, C6 to C5, C7 to C6, C8 to C7, C9 to C8, C10 to C9, D11 to D10, D12 to D11, D13 to D12, D14 to D13, D15 to D14, D3 to D2, D4 to D3, D5 to D4, D6 to D5, D7 to D6, D8 to D7, D9 to D8, D10 to D9
Connections:
- net +3V3: now also SW8va1.1 (A), SW8vb1.1 (A), SWA1.1 (A), SWB1.1 (A), SWBb1.1 (A), SWC1.1 (A), SWCTRL1.1 (A), SWD1.1 (A), SWDup1.1 (A), SWE1.1 (A), SWEb1.1 (A), SWF1.1 (A), SWG1.1 (A), SWGs1.1 (A), SWSPR1.1 (A)
- net +5V: now also C11.1, C12.1, C13.1, C14.1, C15.1, C16.1, C17.1, C4.1, C5.1, C6.1, C7.1, C8.1, C9.1, D10.2 (AVDD), D11.2 (AVDD), D12.2 (AVDD), D13.2 (AVDD), D14.2 (AVDD), D2.2 (AVDD), D3.2 (AVDD), D4.2 (AVDD), D5.2 (AVDD), D6.2 (AVDD), D7.2 (AVDD), D8.2 (AVDD), D9.2 (AVDD)
- net 8va: now also SW8va1.2 (B)
- net 8vb: now also SW8vb1.2 (B)
- net A: now also SWA1.2 (B)
- net B: now also SWB1.2 (B)
- net Bb: now also SWBb1.2 (B)
- net C: now also SWC1.2 (B)
- net Ctrl: now also SWCTRL1.2 (B)
- net D: now also SWD1.2 (B)
- net Dup: now also SWDup1.2 (B)
- net E: now also SWE1.2 (B)
- net Eb: now also SWEb1.2 (B)
- net F: now also SWF1.2 (B)
- net G: now also SWG1.2 (B)
- net Gs: now also SWGs1.2 (B)
- net Spr: now also SWSPR1.2 (B)
- net at D14.3 (DIn): now also D2.1 (DOut)
- removed net VSYS: A1.39 (VSYS), C11.1, C12.1, C13.1, C14.1, C15.1, C16.1, C17.1, C4.1, C5.1, C6.1, C7.1, C8.1, C9.1, D1.1 (K), D10.2 (AVDD), D11.2 (AVDD), D12.2 (AVDD), D13.2 (AVDD), D14.2 (AVDD), D2.2 (AVDD), D3.2 (AVDD), D4.2 (AVDD), D5.2 (AVDD), D6.2 (AVDD), D7.2 (AVDD), D8.2 (AVDD), D9.2 (AVDD), J4.19
- new net: A1.39 (VSYS), D1.1 (K), J4.19
