File: pcb/PicoSax/PicoSax.kicad_sch (KiCad schematic)
At the start: 75 parts, among them J3 Conn_01x02, SW8va1 Gateron_KS-33, SW8vb1 Gateron_KS-33, U1 Perfboard

Commit message: Partial Route
Parts:
- added R20, R21, R22: 0, Resistor_SMD:R_0805_2012Metric_Pad1.20x1.40mm_HandSolder, symbol Device:R
Connections:
- net +3V3: now also SWC1.2 (B), SWD1.2 (B), SWDup1.2 (B), SWE1.2 (B), SWEb1.2 (B), SWF1.2 (B); no longer SWC1.1 (A), SWD1.1 (A), SWDup1.1 (A), SWE1.1 (A), SWEb1.1 (A), SWF1.1 (A)
- net +5V: now also R20.1
- net C: now also SWC1.1 (A); no longer SWC1.2 (B)
- net D: now also SWD1.1 (A); no longer SWD1.2 (B)
- net Dup: now also SWDup1.1 (A); no longer SWDup1.2 (B)
- net E: now also SWE1.1 (A); no longer SWE1.2 (B)
- net Eb: now also SWEb1.1 (A); no longer SWEb1.2 (B)
- net F: now also SWF1.1 (A); no longer SWF1.2 (B)
- net VSYS: now also R21.1; no longer C10.1, C12.1, C13.1, C14.1, C15.1, C16.1, C17.1, C18.1, C4.1, C5.1, C6.1, C7.1, C8.1, C9.1, D10.2 (AVDD), D11.2 (AVDD), D12.2 (AVDD), D13.2 (AVDD), D14.2 (AVDD), D15.2 (AVDD), D2.2 (AVDD), D3.2 (AVDD), D4.2 (AVDD), D5.2 (AVDD), D6.2 (AVDD), D7.2 (AVDD), D8.2 (AVDD), D9.2 (AVDD)
- new net VLED: C10.1, C12.1, C13.1, C14.1, C15.1, C16.1, C17.1, C18.1, C4.1, C5.1, C6.1, C7.1, C8.1, C9.1, D10.2 (AVDD), D11.2 (AVDD), D12.2 (AVDD), D13.2 (AVDD), D14.2 (AVDD), D15.2 (AVDD), D2.2 (AVDD), D3.2 (AVDD), D4.2 (AVDD), D5.2 (AVDD), D6.2 (AVDD), D7.2 (AVDD), D8.2 (AVDD), D9.2 (AVDD), R20.2, R21.2, R22.2
- no-connect marks 1 -> 2
Other:
- moved on the sheet: SWC1, SWD1, SWDup1, SWE1, SWEb1, SWF1

Commit message: V2 ready
Other:
- note added: "Ability to choose or apply different voltage to power LEDs"
- note added: "Choice of breath sensor MP3V5004GP or BPS110 AD0P15"
- moved on the sheet: C1, C10, C11, C12, C13, C14, C15, C16, C17, C18, C2, C3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
